Commit message: added tcp link

File: zimmer_gp406n/urdf/gripper.urdf.xacro (robot description, xacro)
@@ -26,4 +26,10 @@
         </link>
 <!--        TODO -  add EE-link-->
+        <link name="${prefix}tcp_link"/>
+        <joint name="${prefix}tcp_joint" type="fixed">
+            <origin xyz="0.107 0 -0.032" rpy="0 0.5 0"/>
+            <parent link="${parent}"/>
+            <child link="${prefix}tcp_link"/>
+        </joint>
     </xacro:macro>
 </robot>

Commit message: gripper orientation fixed

File: zimmer_gp406n/urdf/gripper.urdf.xacro (robot description, xacro)
@@ -28,5 +28,5 @@
         <link name="${prefix}tcp_link"/>
         <joint name="${prefix}tcp_joint" type="fixed">
-            <origin xyz="0.107 0 -0.032" rpy="0 0.5 0"/>
+            <origin xyz="0.107 0 -0.032" rpy="0 2.07079632679 0"/>
             <parent link="${parent}"/>
             <child link="${prefix}tcp_link"/>
