Commit message: lowered roof collision object to avoid collisions with the camera

File: kuka_kr3_cell_description/urdf/cell.urdf.xacro (robot description, xacro)
@@ -81,5 +81,5 @@
         </link>
         <joint name="{prefix}roof_joint" type="fixed">
-            <origin xyz="0 0 0.84" rpy="0 0 0"/>
+            <origin xyz="0 0 0.64" rpy="0 0 0"/>
             <parent link="${prefix}cell_link"/>
             <child link="${prefix}roof"/>
