Commit message: Add publishing srdf file

File: kuka_kr10r1100sixx_cell_description/urdf/kr10_cylinder.xacro (robot description, xacro)
@@ -1,16 +1,16 @@
 <?xml version="1.0"?>
 <robot name="kuka_kr10_cell" xmlns:xacro="http://wiki.ros.org/xacro">
-    <xacro:include filename="$(find kuka_kr10r1100sixx_cell_description)/urdf/kr10_cylinder_macro.xacro"/>
-    <xacro:include filename="$(find kuka_kr10r1100sixx_cell_description)/urdf/kr10_macro.ros2_control.xacro"/>
-    <xacro:arg name="initial_positions_file" default="$(find kuka_kr10r1100sixx_cell_description)/config/initial_positions.yaml"/>
-    <xacro:arg name="robot_ip" default="10.181.116.41"/>
-    <xacro:arg name="robot_port" default="54600"/>
-    <xacro:arg name="use_fake_hardware" default="true"/>
+    <xacro:include filename="$(find kuka_kr10r1100sixx_cell_description)/urdf/kr10_cylinder_macro.xacro" />
+    <xacro:include filename="$(find kuka_kr10r1100sixx_cell_description)/urdf/kr10_macro.ros2_control.xacro" />
+    <xacro:arg name="initial_positions_file" default="$(find kuka_kr10r1100sixx_cell_description)/config/initial_positions.yaml" />
+    <xacro:arg name="robot_ip" default="10.181.116.41" />
+    <xacro:arg name="eki_robot_port" default="54600" />
+    <xacro:arg name="use_fake_hardware" default="true" />
     <xacro:kuka_kr10r1100sixx prefix="" initial_positions_file="$(arg initial_positions_file)"
-                              robot_ip="$(arg robot_ip)" robot_port="$(arg robot_port)"
-                              use_fake_hardware="$(arg use_fake_hardware)"/>
+        robot_ip="$(arg robot_ip)" eki_robot_port="$(arg eki_robot_port)"
+        use_fake_hardware="$(arg use_fake_hardware)" />
     <xacro:kr10_gripper_ros2_control
-    name="gripper_control"
-    prefix=""
-    use_fake_hardware="$(arg use_fake_hardware)" />
+        name="gripper_control"
+        prefix=""
+        use_fake_hardware="$(arg use_fake_hardware)" />
 </robot>

File: kuka_kr10r1100sixx_cell_description/urdf/kr10_cylinder_macro.xacro (robot description, xacro)
@@ -1,21 +1,21 @@
 <?xml version="1.0"?>
 <robot xmlns:xacro="http://wiki.ros.org/xacro">
-    <xacro:include filename="$(find kuka_common)/urdf/common_constants.xacro"/>
-    <xacro:include filename="$(find kuka_common)/urdf/common_materials.xacro"/>
-    <xacro:include filename="$(find kuka_common)/urdf/kuka.ros2_control.xacro"/>
-    <xacro:include filename="$(find kuka_kr10r1100sixx_cell_description)/urdf/kr10_macro.ros2_control.xacro"/>
-    <xacro:macro name="kuka_kr10r1100sixx" params="prefix initial_positions_file robot_ip robot_port use_fake_hardware">
+    <xacro:include filename="$(find kuka_common)/urdf/common_constants.xacro" />
+    <xacro:include filename="$(find kuka_common)/urdf/common_materials.xacro" />
+    <xacro:include filename="$(find kuka_common)/urdf/kuka.ros2_control.xacro" />
+    <xacro:include filename="$(find kuka_kr10r1100sixx_cell_description)/urdf/kr10_macro.ros2_control.xacro" />
+    <xacro:macro name="kuka_kr10r1100sixx" params="prefix initial_positions_file robot_ip eki_robot_port use_fake_hardware">
         <link name="${prefix}table_link">
             <visual>
-                <origin xyz="0 0 0" rpy="0 0 0"/>
-                <geometry>
-                    <mesh filename="package://kuka_kr10r1100sixx_cell_description/meshes/kr10r1100sixx_cell/visual/table0.001.stl"/>
-                </geometry>
-                <xacro:material_kuka_ral_silver_gray/>
-            </visual>
-            <collision>
-                <origin xyz="0 0 0" rpy="0 0 0"/>
-                <geometry>
-                    <mesh filename="package://kuka_kr10r1100sixx_cell_description/meshes/kr10r1100sixx_cell/collision/table0.001.stl"/>
+                <origin xyz="0 0 0" rpy="0 0 0" />
+                <geometry>
+                    <mesh filename="package://kuka_kr10r1100sixx_cell_description/meshes/kr10r1100sixx_cell/visual/table0.001.stl" />
+                </geometry>
+                <xacro:material_kuka_ral_silver_gray />
+            </visual>
+            <collision>
+                <origin xyz="0 0 0" rpy="0 0 0" />
+                <geometry>
+                    <mesh filename="package://kuka_kr10r1100sixx_cell_description/meshes/kr10r1100sixx_cell/collision/table0.001.stl" />
                 </geometry>
             </collision>
@@ -23,14 +23,14 @@
         <link name="${prefix}base_link">
             <visual>
-                <origin xyz="0 0 0" rpy="0 0 0"/>
-                <geometry>
-                    <mesh filename="package://kuka_kr10_description/meshes/kr10r1100sixx/visual/base_link.stl"/>
-                </geometry>
-                <xacro:material_kuka_black/>
-            </visual>
-            <collision>
-                <origin xyz="0 0 0" rpy="0 0 0"/>
-                <geometry>
-                    <mesh filename="package://kuka_kr10_description/meshes/kr10r1100sixx/collision/base_link.stl"/>
+                <origin xyz="0 0 0" rpy="0 0 0" />
+                <geometry>
+                    <mesh filename="package://kuka_kr10_description/meshes/kr10r1100sixx/visual/base_link.stl" />
+                </geometry>
+                <xacro:material_kuka_black />
+            </visual>
+            <collision>
+                <origin xyz="0 0 0" rpy="0 0 0" />
+                <geometry>
+                    <mesh filename="package://kuka_kr10_description/meshes/kr10r1100sixx/collision/base_link.stl" />
                 </geometry>
             </collision>
@@ -38,14 +38,14 @@
         <link name="${prefix}link_1">
             <visual>
-                <origin xyz="0 0 0" rpy="0 0 0"/>
-                <geometry>
-                    <mesh filename="package://kuka_kr10_description/meshes/kr10r1100sixx/visual/link_1.stl"/>
-                </geometry>
-                <xacro:material_kuka_orange/>
-            </visual>
-            <collision>
-                <origin xyz="0 0 0" rpy="0 0 0"/>
-                <geometry>
-                    <mesh filename="package://kuka_kr10_description/meshes/kr10r1100sixx/collision/link_1.stl"/>
+                <origin xyz="0 0 0" rpy="0 0 0" />
+                <geometry>
+                    <mesh filename="package://kuka_kr10_description/meshes/kr10r1100sixx/visual/link_1.stl" />
+                </geometry>
+                <xacro:material_kuka_orange />
+            </visual>
+            <collision>
+                <origin xyz="0 0 0" rpy="0 0 0" />
+                <geometry>
+                    <mesh filename="package://kuka_kr10_description/meshes/kr10r1100sixx/collision/link_1.stl" />
                 </geometry>
             </collision>
@@ -53,14 +53,14 @@
         <link name="${prefix}link_2">
             <visual>
-                <origin xyz="0 0 0" rpy="0 0 0"/>
-                <geometry>
-                    <mesh filename="package://kuka_kr10_description/meshes/kr10r1100sixx/visual/link_2.stl"/>
-                </geometry>
-                <xacro:material_kuka_orange/>
-            </visual>
-            <collision>
-                <origin xyz="0 0 0" rpy="0 0 0"/>
-                <geometry>
-                    <mesh filename="package://kuka_kr10_description/meshes/kr10r1100sixx/collision/link_2.stl"/>
+                <origin xyz="0 0 0" rpy="0 0 0" />
+                <geometry>
+                    <mesh filename="package://kuka_kr10_description/meshes/kr10r1100sixx/visual/link_2.stl" />
+                </geometry>
+                <xacro:material_kuka_orange />
+            </visual>
+            <collision>
+                <origin xyz="0 0 0" rpy="0 0 0" />
+                <geometry>
+                    <mesh filename="package://kuka_kr10_description/meshes/kr10r1100sixx/collision/link_2.stl" />
                 </geometry>
             </collision>
@@ -68,14 +68,14 @@
         <link name="${prefix}link_3">
             <visual>
-                <origin xyz="0 0 0" rpy="0 0 0"/>
-                <geometry>
-                    <mesh filename="package://kuka_kr10_description/meshes/kr10r1100sixx/visual/link_3.stl"/>
-                </geometry>
-                <xacro:material_kuka_orange/>
-            </visual>
-            <collision>
-                <origin xyz="0 0 0" rpy="0 0 0"/>
-                <geometry>
-                    <mesh filename="package://kuka_kr10_description/meshes/kr10r1100sixx/collision/link_3.stl"/>
+                <origin xyz="0 0 0" rpy="0 0 0" />
+                <geometry>
+                    <mesh filename="package://kuka_kr10_description/meshes/kr10r1100sixx/visual/link_3.stl" />
+                </geometry>
+                <xacro:material_kuka_orange />
+            </visual>
+            <collision>
+                <origin xyz="0 0 0" rpy="0 0 0" />
+                <geometry>
+                    <mesh filename="package://kuka_kr10_description/meshes/kr10r1100sixx/collision/link_3.stl" />
                 </geometry>
             </collision>
@@ -83,14 +83,14 @@
         <link name="${prefix}link_4">
             <visual>
-                <origin xyz="0 0 0" rpy="0 0 0"/>
-                <geometry>
-                    <mesh filename="package://kuka_kr10_description/meshes/kr10r1100sixx/visual/link_4.stl"/>
-                </geometry>
-                <xacro:material_kuka_orange/>
-            </visual>
-            <collision>
-                <origin xyz="0 0 0" rpy="0 0 0"/>
-                <geometry>
-                    <mesh filename="package://kuka_kr10_description/meshes/kr10r1100sixx/collision/link_4.stl"/>
+                <origin xyz="0 0 0" rpy="0 0 0" />
+                <geometry>
+                    <mesh filename="package://kuka_kr10_description/meshes/kr10r1100sixx/visual/link_4.stl" />
+                </geometry>
+                <xacro:material_kuka_orange />
+            </visual>
+            <collision>
+                <origin xyz="0 0 0" rpy="0 0 0" />
+                <geometry>
+                    <mesh filename="package://kuka_kr10_description/meshes/kr10r1100sixx/collision/link_4.stl" />
                 </geometry>
             </collision>
@@ -98,14 +98,14 @@
         <link name="${prefix}link_5">
             <visual>
-                <origin xyz="0 0 0" rpy="0 0 0"/>
-                <geometry>
-                    <mesh filename="package://kuka_kr10_description/meshes/kr10r1100sixx/visual/link_5.stl"/>
-                </geometry>
-                <xacro:material_kuka_orange/>
-            </visual>
-            <collision>
-                <origin xyz="0 0 0" rpy="0 0 0"/>
-                <geometry>
-                    <mesh filename="package://kuka_kr10_description/meshes/kr10r1100sixx/collision/link_5.stl"/>
+                <origin xyz="0 0 0" rpy="0 0 0" />
+                <geometry>
+                    <mesh filename="package://kuka_kr10_description/meshes/kr10r1100sixx/visual/link_5.stl" />
+                </geometry>
+                <xacro:material_kuka_orange />
+            </visual>
+            <collision>
+                <origin xyz="0 0 0" rpy="0 0 0" />
+                <geometry>
+                    <mesh filename="package://kuka_kr10_description/meshes/kr10r1100sixx/collision/link_5.stl" />
                 </geometry>
             </collision>
@@ -113,14 +113,14 @@
         <link name="${prefix}link_6">
             <visual>
-                <origin xyz="0 0 0" rpy="0 0 0"/>
-                <geometry>
-                    <mesh filename="package://kuka_kr10_description/meshes/kr10r1100sixx/visual/link_6.stl"/>
-                </geometry>
-                <xacro:material_kuka_pedestal/>
-            </visual>
-            <collision>
-                <origin xyz="0 0 0" rpy="0 0 0"/>
-                <geometry>
-                    <mesh filename="package://kuka_kr10_description/meshes/kr10r1100sixx/collision/link_6.stl"/>
+                <origin xyz="0 0 0" rpy="0 0 0" />
+                <geometry>
+                    <mesh filename="package://kuka_kr10_description/meshes/kr10r1100sixx/visual/link_6.stl" />
+                </geometry>
+                <xacro:material_kuka_pedestal />
+            </visual>
+            <collision>
+                <origin xyz="0 0 0" rpy="0 0 0" />
+                <geometry>
+                    <mesh filename="package://kuka_kr10_description/meshes/kr10r1100sixx/collision/link_6.stl" />
                 </geometry>
             </collision>
@@ -128,14 +128,14 @@
         <link name="${prefix}shelf">
             <visual>
-                <origin xyz="0 0 0" rpy="0 0 0"/>
-                <geometry>
-                    <mesh filename="package://kuka_kr10r1100sixx_cell_description/meshes/kr10r1100sixx_cell/visual/shelf_new.stl"/>
-                </geometry>
-                <xacro:material_kuka_ral_silver_gray/>
-            </visual>
-            <collision>
-                <origin xyz="0 0 0" rpy="0 0 0"/>
-                <geometry>
-                    <mesh filename="package://kuka_kr10r1100sixx_cell_description/meshes/kr10r1100sixx_cell/collision/shelf_new.stl"/>
+                <origin xyz="0 0 0" rpy="0 0 0" />
+                <geometry>
+                    <mesh filename="package://kuka_kr10r1100sixx_cell_description/meshes/kr10r1100sixx_cell/visual/shelf_new.stl" />
+                </geometry>
+                <xacro:material_kuka_ral_silver_gray />
+            </visual>
+            <collision>
+                <origin xyz="0 0 0" rpy="0 0 0" />
+                <geometry>
+                    <mesh filename="package://kuka_kr10r1100sixx_cell_description/meshes/kr10r1100sixx_cell/collision/shelf_new.stl" />
                 </geometry>
             </collision>
@@ -144,14 +144,14 @@
         <link name="${prefix}gripper_base">
             <visual>
-                <origin xyz="0 0 0" rpy="0 ${radians(180)} ${radians(270)}"/>
-                <geometry>
-                    <mesh filename="package://kuka_kr10r1100sixx_cell_description/meshes/kr10r1100sixx_cell/visual/gripper_visual_base.stl"/>
-                </geometry>
-                <xacro:material_kuka_ral_silver_gray/>
-            </visual>
-            <collision>
-                <origin xyz="0 0 0" rpy="0 ${radians(180)} ${radians(270)}"/>
-                <geometry>
-                    <mesh filename="package://kuka_kr10r1100sixx_cell_description/meshes/kr10r1100sixx_cell/collision/gripper_col_base.stl"/>
+                <origin xyz="0 0 0" rpy="0 ${radians(180)} ${radians(270)}" />
+                <geometry>
+                    <mesh filename="package://kuka_kr10r1100sixx_cell_description/meshes/kr10r1100sixx_cell/visual/gripper_visual_base.stl" />
+                </geometry>
+                <xacro:material_kuka_ral_silver_gray />
+            </visual>
+            <collision>
+                <origin xyz="0 0 0" rpy="0 ${radians(180)} ${radians(270)}" />
+                <geometry>
+                    <mesh filename="package://kuka_kr10r1100sixx_cell_description/meshes/kr10r1100sixx_cell/collision/gripper_col_base.stl" />
                 </geometry>
             </collision>
@@ -159,14 +159,14 @@
         <link name="${prefix}cylinder_back_left">
             <visual>
-                <origin xyz="0 0 0" rpy="0 ${radians(180)} ${radians(270)}"/>
-                <geometry>
-                    <mesh filename="package://kuka_kr10r1100sixx_cell_description/meshes/kr10r1100sixx_cell/visual/cylinder_back_left.stl"/>
-                </geometry>
-                <xacro:material_kuka_ral_silver_gray/>
-            </visual>
-            <collision>
-                <origin xyz="0 0 0" rpy="0 ${radians(180)} ${radians(270)}"/>
-                <geometry>
-                    <mesh filename="package://kuka_kr10r1100sixx_cell_description/meshes/kr10r1100sixx_cell/collision/cylinder_col_bl.stl"/>
+                <origin xyz="0 0 0" rpy="0 ${radians(180)} ${radians(270)}" />
+                <geometry>
+                    <mesh filename="package://kuka_kr10r1100sixx_cell_description/meshes/kr10r1100sixx_cell/visual/cylinder_back_left.stl" />
+                </geometry>
+                <xacro:material_kuka_ral_silver_gray />
+            </visual>
+            <collision>
+                <origin xyz="0 0 0" rpy="0 ${radians(180)} ${radians(270)}" />
+                <geometry>
+                    <mesh filename="package://kuka_kr10r1100sixx_cell_description/meshes/kr10r1100sixx_cell/collision/cylinder_col_bl.stl" />
                 </geometry>
             </collision>
@@ -174,14 +174,14 @@
         <link name="${prefix}cylinder_back_right">
             <visual>
-                <origin xyz="0 0 0" rpy="0 ${radians(180)} ${radians(270)}"/>
-                <geometry>
-                    <mesh filename="package://kuka_kr10r1100sixx_cell_description/meshes/kr10r1100sixx_cell/visual/cylinder_back_right.stl"/>
-                </geometry>
-                <xacro:material_kuka_ral_silver_gray/>
-            </visual>
-            <collision>
-                <origin xyz="0 0 0" rpy="0 ${radians(180)} ${radians(270)}"/>
-                <geometry>
-                    <mesh filename="package://kuka_kr10r1100sixx_cell_description/meshes/kr10r1100sixx_cell/collision/cylinder_col_br.stl"/>
+                <origin xyz="0 0 0" rpy="0 ${radians(180)} ${radians(270)}" />
+                <geometry>
+                    <mesh filename="package://kuka_kr10r1100sixx_cell_description/meshes/kr10r1100sixx_cell/visual/cylinder_back_right.stl" />
+                </geometry>
+                <xacro:material_kuka_ral_silver_gray />
+            </visual>
+            <collision>
+                <origin xyz="0 0 0" rpy="0 ${radians(180)} ${radians(270)}" />
+                <geometry>
+                    <mesh filename="package://kuka_kr10r1100sixx_cell_description/meshes/kr10r1100sixx_cell/collision/cylinder_col_br.stl" />
                 </geometry>
             </collision>
@@ -189,14 +189,14 @@
         <link name="${prefix}cylinder_front_left">
             <visual>
-                <origin xyz="0 0 0" rpy="0 ${radians(180)} ${radians(270)}"/>
-                <geometry>
-                    <mesh filename="package://kuka_kr10r1100sixx_cell_description/meshes/kr10r1100sixx_cell/visual/cylinder_front_left.stl"/>
-                </geometry>
-                <xacro:material_kuka_ral_silver_gray/>
-            </visual>
-            <collision>
-                <origin xyz="0 0 0" rpy="0 ${radians(180)} ${radians(270)}"/>
-                <geometry>
-                    <mesh filename="package://kuka_kr10r1100sixx_cell_description/meshes/kr10r1100sixx_cell/collision/cylinder_col_fl.stl"/>
+                <origin xyz="0 0 0" rpy="0 ${radians(180)} ${radians(270)}" />
+                <geometry>
+                    <mesh filename="package://kuka_kr10r1100sixx_cell_description/meshes/kr10r1100sixx_cell/visual/cylinder_front_left.stl" />
+                </geometry>
+                <xacro:material_kuka_ral_silver_gray />
+            </visual>
+            <collision>
+                <origin xyz="0 0 0" rpy="0 ${radians(180)} ${radians(270)}" />
+                <geometry>
+                    <mesh filename="package://kuka_kr10r1100sixx_cell_description/meshes/kr10r1100sixx_cell/collision/cylinder_col_fl.stl" />
                 </geometry>
             </collision>
@@ -204,164 +204,164 @@
         <link name="${prefix}cylinder_front_right">
             <visual>
-                <origin xyz="0 0 0" rpy="0 ${radians(180)} ${radians(270)}"/>
-                <geometry>
-                    <mesh filename="package://kuka_kr10r1100sixx_cell_description/meshes/kr10r1100sixx_cell/visual/cylinder_front_right.stl"/>
-                </geometry>
-                <xacro:material_kuka_ral_silver_gray/>
-            </visual>
-            <collision>
-                <origin xyz="0 0 0" rpy="0 ${radians(180)} ${radians(270)}"/>
-                <geometry>
-                    <mesh filename="package://kuka_kr10r1100sixx_cell_description/meshes/kr10r1100sixx_cell/collision/cylinder_col_fr.stl"/>
-                </geometry>
-            </collision>
-        </link>
-        <link name="${prefix}tcp"/>
-        <link name="${prefix}tcp_1"/>
-        <link name="${prefix}tcp_2"/>
-        <link name="${prefix}tcp_3"/>
-        <link name="${prefix}tcp_4"/>
-        <link name="${prefix}tcp_5"/>
-        <link name="${prefix}tcp_6"/>
-        <link name="${prefix}tcp_7"/>
+                <origin xyz="0 0 0" rpy="0 ${radians(180)} ${radians(270)}" />
+                <geometry>
+                    <mesh filename="package://kuka_kr10r1100sixx_cell_description/meshes/kr10r1100sixx_cell/visual/cylinder_front_right.stl" />
+                </geometry>
+                <xacro:material_kuka_ral_silver_gray />
+            </visual>
+            <collision>
+                <origin xyz="0 0 0" rpy="0 ${radians(180)} ${radians(270)}" />
+                <geometry>
+                    <mesh filename="package://kuka_kr10r1100sixx_cell_description/meshes/kr10r1100sixx_cell/collision/cylinder_col_fr.stl" />
+                </geometry>
+            </collision>
+        </link>
+        <link name="${prefix}tcp" />
+        <link name="${prefix}tcp_1" />
+        <link name="${prefix}tcp_2" />
+        <link name="${prefix}tcp_3" />
+        <link name="${prefix}tcp_4" />
+        <link name="${prefix}tcp_5" />
+        <link name="${prefix}tcp_6" />
+        <link name="${prefix}tcp_7" />
         <joint name="${prefix}joint_a0" type="fixed">
-            <parent link="${prefix}table_link"/>
-            <child link="${prefix}base_link"/>
-            <origin xyz="0.2 0.4 0.965" rpy="0 0 0"/>
+            <parent link="${prefix}table_link" />
+            <child link="${prefix}base_link" />
+            <origin xyz="0.2 0.4 0.965" rpy="0 0 0" />
         </joint>
         <joint name="${prefix}joint_a1" type="revolute">
-            <origin xyz="0 0 0.400" rpy="0 0 0"/>
-            <parent link="${prefix}base_link"/>
-            <child link="${prefix}link_1"/>
-            <axis xyz="0 0 -1"/>
-            <limit effort="0" lower="${radians(-170)}" upper="${radians(170)}" velocity="${radians(300)}"/>
+            <origin xyz="0 0 0.400" rpy="0 0 0" />
+            <parent link="${prefix}base_link" />
+            <child link="${prefix}link_1" />
+            <axis xyz="0 0 -1" />
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