Commit message: Refactor container xmls. container.xacro is loaded with different origins and a name parameter. Move meshes to correct folder.

File: kuka_kr10r1100sixx_cell_description/urdf/aip_cell_macro.xacro (robot description, xacro)
@@ -8,5 +8,5 @@
                 <origin xyz="0 0 0" rpy="0 0 0"/>
                 <geometry>
-                    <mesh filename="package://kuka_kr10r1100sixx_cell_description/meshes/kr10r1100sixx_cell/visual/table0.001.stl"/>
+                    <mesh filename="package://kuka_kr10r1100sixx_cell_description/meshes/aip_cell/visual/table0.001.stl"/>
                 </geometry>
                 <xacro:material_kuka_ral_silver_gray/>
@@ -15,5 +15,5 @@
                 <origin xyz="0 0 0" rpy="0 0 0"/>
                 <geometry>
-                    <mesh filename="package://kuka_kr10r1100sixx_cell_description/meshes/kr10r1100sixx_cell/collision/table0.001.stl"/>
+                    <mesh filename="package://kuka_kr10r1100sixx_cell_description/meshes/aip_cell/collision/table0.001.stl"/>
                 </geometry>
             </collision>
@@ -23,5 +23,5 @@
                 <origin xyz="0 0 0" rpy="0 0 0"/>
                 <geometry>
-                    <mesh filename="package://kuka_kr10r1100sixx_cell_description/meshes/kr10r1100sixx_cell/visual/shelf_new.stl"/>
+                    <mesh filename="package://kuka_kr10r1100sixx_cell_description/meshes/aip_cell/visual/shelf_new.stl"/>
                 </geometry>
                 <xacro:material_kuka_ral_silver_gray/>
@@ -30,5 +30,5 @@
                 <origin xyz="0 0 0" rpy="0 0 0"/>
                 <geometry>
-                    <mesh filename="package://kuka_kr10r1100sixx_cell_description/meshes/kr10r1100sixx_cell/collision/shelf_new.stl"/>
+                    <mesh filename="package://kuka_kr10r1100sixx_cell_description/meshes/aip_cell/collision/shelf_new.stl"/>
                 </geometry>
             </collision>
