Commit message: Rename package to aip_cell_description

File: aip_cell_description/urdf/aip_cell_macro.xacro (robot description, xacro)
@@ -8,5 +8,5 @@
                 <origin xyz="0 0 0" rpy="0 0 0"/>
                 <geometry>
-                    <mesh filename="package://kuka_kr10r1100sixx_cell_description/meshes/aip_cell/visual/table0.001.stl"/>
+                    <mesh filename="package://aip_cell_description/meshes/aip_cell/visual/table0.001.stl"/>
                 </geometry>
                 <xacro:material_kuka_ral_silver_gray/>
@@ -15,5 +15,5 @@
                 <origin xyz="0 0 0" rpy="0 0 0"/>
                 <geometry>
-                    <mesh filename="package://kuka_kr10r1100sixx_cell_description/meshes/aip_cell/collision/table0.001.stl"/>
+                    <mesh filename="package://aip_cell_description/meshes/aip_cell/collision/table0.001.stl"/>
                 </geometry>
             </collision>
@@ -23,5 +23,5 @@
                 <origin xyz="0 0 0" rpy="0 0 0"/>
                 <geometry>
-                    <mesh filename="package://kuka_kr10r1100sixx_cell_description/meshes/aip_cell/visual/shelf_new.stl"/>
+                    <mesh filename="package://aip_cell_description/meshes/aip_cell/visual/shelf_new.stl"/>
                 </geometry>
                 <xacro:material_kuka_ral_silver_gray/>
@@ -30,5 +30,5 @@
                 <origin xyz="0 0 0" rpy="0 0 0"/>
                 <geometry>
-                    <mesh filename="package://kuka_kr10r1100sixx_cell_description/meshes/aip_cell/collision/shelf_new.stl"/>
+                    <mesh filename="package://aip_cell_description/meshes/aip_cell/collision/shelf_new.stl"/>
                 </geometry>
             </collision>

File: aip_cell_description/urdf/aip_kr10_cell.xacro (robot description, xacro)
@@ -1,8 +1,8 @@
 <?xml version="1.0"?>
 <robot name="aip_kr10_cell" xmlns:xacro="http://wiki.ros.org/xacro">
-    <xacro:include filename="$(find kuka_kr10r1100sixx_cell_description)/urdf/aip_cell_macro.xacro"/>
+    <xacro:include filename="$(find aip_cell_description)/urdf/aip_cell_macro.xacro"/>
     <xacro:include filename="$(find aip_bosch_gripper)/urdf/gripper_macro.xacro"/>
     <xacro:include filename="$(find kuka_kr10_description)/urdf/kr10r1100sixx_macro.xacro"/>
-    <xacro:arg name="initial_positions_file" default="$(find kuka_kr10r1100sixx_cell_description)/config/initial_positions.yaml"/>
+    <xacro:arg name="initial_positions_file" default="$(find aip_cell_description)/config/initial_positions.yaml"/>
     <xacro:arg name="robot_ip" default="10.166.32.145"/>
     <xacro:arg name="eki_robot_port" default="54600"/>

File: aip_cell_description/urdf/aip_kr10_container_cell.xacro (robot description, xacro)
@@ -1,9 +1,9 @@
 <?xml version="1.0"?>
 <robot name="aip_kr10_cell" xmlns:xacro="http://wiki.ros.org/xacro">
-    <xacro:include filename="$(find kuka_kr10r1100sixx_cell_description)/urdf/aip_cell_macro.xacro"/>
+    <xacro:include filename="$(find aip_cell_description)/urdf/aip_cell_macro.xacro"/>
     <xacro:include filename="$(find aip_bosch_gripper)/urdf/gripper_macro.xacro"/>
     <xacro:include filename="$(find kuka_kr10_description)/urdf/kr10r1100sixx_macro.xacro"/>
-    <xacro:include filename="$(find kuka_kr10r1100sixx_cell_description)/urdf/container_macro.xacro"/>
-    <xacro:arg name="initial_positions_file" default="$(find kuka_kr10r1100sixx_cell_description)/config/initial_positions.yaml"/>
+    <xacro:include filename="$(find aip_cell_description)/urdf/container_macro.xacro"/>
+    <xacro:arg name="initial_positions_file" default="$(find aip_cell_description)/config/initial_positions.yaml"/>
     <xacro:arg name="robot_ip" default="10.166.32.145"/>
     <xacro:arg name="eki_robot_port" default="54600"/>

File: aip_cell_description/urdf/container_macro.xacro (robot description, xacro)
@@ -8,5 +8,5 @@
                 <origin xyz="0 0 0" rpy="0 0 0"/>
                 <geometry>
-                    <mesh filename="package://kuka_kr10r1100sixx_cell_description/meshes/bosch_container/visual/container_${number}.stl"/>
+                    <mesh filename="package://aip_cell_description/meshes/bosch_container/visual/container_${number}.stl"/>
                 </geometry>
                 <xacro:material_kuka_ral_pearly_white/>
@@ -15,5 +15,5 @@
                 <origin xyz="0 0 0" rpy="0 0 0"/>
                 <geometry>
-                    <mesh filename="package://kuka_kr10r1100sixx_cell_description/meshes/bosch_container/collision/container_${number}.stl"/>
+                    <mesh filename="package://aip_cell_description/meshes/bosch_container/collision/container_${number}.stl"/>
                 </geometry>
             </collision>

Commit message: Add new STL files for visual and collision meshes, and update xacro files

File: aip_cell_description/urdf/aip_cell_macro.xacro (robot description, xacro)
@@ -8,5 +8,12 @@
                 <origin xyz="0 0 0" rpy="0 0 0"/>
                 <geometry>
-                    <mesh filename="package://aip_cell_description/meshes/aip_cell/visual/table0.001.stl"/>
+                    <mesh filename="package://aip_cell_description/meshes/aip_cell/visual/table0.001.stl" scale="0.001 0.001 0.001"/>
+                </geometry>
+                <xacro:material_kuka_ral_silver_gray/>
+            </visual>
+            <visual>
+                <origin xyz="0 0 0" rpy="0 0 0"/>
+                <geometry>
+                    <mesh filename="package://aip_cell_description/meshes/aip_cell/visual/Gestell.stl" scale="0.001 0.001 0.001" />
                 </geometry>
                 <xacro:material_kuka_ral_silver_gray/>
@@ -15,5 +22,11 @@
                 <origin xyz="0 0 0" rpy="0 0 0"/>
                 <geometry>
-                    <mesh filename="package://aip_cell_description/meshes/aip_cell/collision/table0.001.stl"/>
+                    <mesh filename="package://aip_cell_description/meshes/aip_cell/collision/table0.001.stl" scale="0.001 0.001 0.001" />
+                </geometry>
+            </collision>
+            <collision>
+                <origin xyz="0 0 0" rpy="0 0 0"/>
+                <geometry>
+                    <mesh filename="package://aip_cell_description/meshes/aip_cell/collision/Gestell.stl" scale="0.001 0.001 0.001" />
                 </geometry>
             </collision>

File: aip_cell_description/urdf/aip_kr10_container_cell.xacro (robot description, xacro)
@@ -46,4 +46,5 @@
         <parent link="$(arg prefix)world"/>
         <child link="$(arg prefix)table_link"/>
+        <child link="$(arg prefix)cell_frame"/>
         <origin xyz="0 0.6 0" rpy="0 0 0"/>
     </joint>

Commit message: Add ejectors visualization

File: aip_cell_description/urdf/aip_cell_macro.xacro (robot description, xacro)
@@ -47,4 +47,19 @@
             </collision>
         </link>
+        <link name="${prefix}ejector">
+            <visual>
+                <origin xyz="0.09 -0.16 0.05" rpy="0 0 0"/>
+                <geometry>
+                    <mesh filename="package://aip_cell_description/meshes/aip_cell/visual/Ejektoren.stl" scale="0.001 0.001 0.001"/>
+                </geometry>
+                <xacro:material_kuka_ral_light_ivory/>
+            </visual>
+            <collision>
+                <origin xyz="0.09 -0.16 0.05" rpy="0 0 0"/>
+                <geometry>
+                    <mesh filename="package://aip_cell_description/meshes/aip_cell/collision/Ejektoren.stl" scale="0.001 0.001 0.001"/>
+                </geometry>
+            </collision>
+        </link>
         <joint name="${prefix}joint_table-shelf" type="fixed">
             <parent link="${prefix}table_link"/>

File: aip_cell_description/urdf/aip_kr10_cell.xacro (robot description, xacro)
@@ -30,3 +30,8 @@
         <origin xyz="0 0 0" rpy="0 0 0"/>
     </joint>
+    <joint name="$(arg prefix)joint_robot-ejector" type="fixed">
+        <parent link="$(arg prefix)link_4"/>
+        <child link="$(arg prefix)ejector"/>
+        <origin xyz="0 0 0" rpy="0 0 0"/>
+    </joint>
 </robot>

Commit message: Add transformation to camera

File: aip_cell_description/urdf/aip_cell_macro.xacro (robot description, xacro)
@@ -15,5 +15,5 @@
                 <origin xyz="0 0 0" rpy="0 0 0"/>
                 <geometry>
-                    <mesh filename="package://aip_cell_description/meshes/aip_cell/visual/Gestell.stl" scale="0.001 0.001 0.001" />
+                    <mesh filename="package://aip_cell_description/meshes/aip_cell/visual/Gestell.stl" scale="0.001 0.001 0.001"/>
                 </geometry>
                 <xacro:material_kuka_ral_silver_gray/>
@@ -22,5 +22,5 @@
                 <origin xyz="0 0 0" rpy="0 0 0"/>
                 <geometry>
-                    <mesh filename="package://aip_cell_description/meshes/aip_cell/collision/table0.001.stl" scale="0.001 0.001 0.001" />
+                    <mesh filename="package://aip_cell_description/meshes/aip_cell/collision/table0.001.stl" scale="0.001 0.001 0.001"/>
                 </geometry>
             </collision>
@@ -28,5 +28,5 @@
                 <origin xyz="0 0 0" rpy="0 0 0"/>
                 <geometry>
-                    <mesh filename="package://aip_cell_description/meshes/aip_cell/collision/Gestell.stl" scale="0.001 0.001 0.001" />
+                    <mesh filename="package://aip_cell_description/meshes/aip_cell/collision/Gestell.stl" scale="0.001 0.001 0.001"/>
                 </geometry>
             </collision>

File: aip_cell_description/urdf/aip_kr10_cell.xacro (robot description, xacro)
@@ -35,3 +35,10 @@
         <origin xyz="0 0 0" rpy="0 0 0"/>
     </joint>
+    <!-- Camera transformation -->
+    <link name="$(arg prefix)camera"/>
+    <joint name="$(arg prefix)table-camera" type="fixed">
+        <parent link="$(arg prefix)table_link"/>
+        <child link="$(arg prefix)camera"/>
+        <origin xyz="0 0 1" rpy="0 0 0"/>
+    </joint>
 </robot>
