Commit message: Approximate camera  pose

File: aip_cell_description/urdf/aip_kr10_cell.xacro (robot description, xacro)
@@ -40,5 +40,5 @@
         <parent link="$(arg prefix)table_link"/>
         <child link="$(arg prefix)camera"/>
-        <origin xyz="0 0 1" rpy="0 0 0"/>
+        <origin xyz="0.7 1 2.1" rpy="0 3.14 0"/>
     </joint>
 </robot>

Commit message: Adapt cell description urdf. Split table and rack

File: aip_cell_description/urdf/aip_kr10_cell.xacro (robot description, xacro)
@@ -1,5 +1,6 @@
 <?xml version="1.0"?>
 <robot name="aip_kr10_cell" xmlns:xacro="http://wiki.ros.org/xacro">
-    <xacro:include filename="$(find aip_cell_description)/urdf/aip_cell_macro.xacro"/>
+    <xacro:include filename="$(find aip_cell_description)/urdf/table_macro.xacro"/>
+    <xacro:include filename="$(find aip_cell_description)/urdf/camera_rack_macro.xacro"/>
     <xacro:include filename="$(find aip_bosch_gripper)/urdf/gripper_macro.xacro"/>
     <xacro:include filename="$(find kuka_kr10_description)/urdf/kr10r1100sixx_macro.xacro"/>
@@ -13,15 +14,21 @@
         use_fake_hardware="$(arg use_fake_hardware)"/>
     <xacro:aip_bosch_gripper prefix="$(arg prefix)"/>
-    <xacro:aip_cell prefix="$(arg prefix)"/>
+    <xacro:table prefix="$(arg prefix)"/>
+    <xacro:camera_rack prefix="$(arg prefix)"/>
     <link name="$(arg prefix)world"/>
-    <joint name="$(arg prefix)joint_world-table" type="fixed">
+    <joint name="$(arg prefix)world-table" type="fixed">
         <parent link="$(arg prefix)world"/>
         <child link="$(arg prefix)table_link"/>
-        <origin xyz="0 0.6 0" rpy="0 0 0"/>
+        <origin xyz="0 0 0" rpy="0 0 0"/>
     </joint>
-    <joint name="$(arg prefix)joint_world-base" type="fixed">
+    <joint name="$(arg prefix)world-rack" type="fixed">
+        <parent link="$(arg prefix)world"/>
+        <child link="$(arg prefix)camera_rack_link"/>
+        <origin xyz="-0.7 0 0" rpy="0 0 0"/>
+    </joint>
+    <joint name="$(arg prefix)world-base" type="fixed">
         <parent link="$(arg prefix)world"/>
         <child link="$(arg prefix)base_link"/>
-        <origin xyz="0.2 1 0.965" rpy="0 0 0"/>
+        <origin xyz="0.2 0.4 0.965" rpy="0 0 0"/>
     </joint>
     <joint name="$(arg prefix)joint_flange-gripper" type="fixed">
@@ -37,8 +44,8 @@
     <!-- Camera transformation -->
     <link name="$(arg prefix)camera"/>
-    <joint name="$(arg prefix)table-camera" type="fixed">
-        <parent link="$(arg prefix)table_link"/>
+    <joint name="$(arg prefix)world-camera" type="fixed">
+        <parent link="$(arg prefix)world"/>
         <child link="$(arg prefix)camera"/>
-        <origin xyz="0.7 1 2.1" rpy="0 3.14 0"/>
+        <origin xyz="0.612 0.954 2.207" rpy="0 3.14 0"/>
     </joint>
 </robot>

File: aip_cell_description/urdf/table_macro.xacro (robot description, xacro)
@@ -3,5 +3,5 @@
     <xacro:include filename="$(find kuka_common)/urdf/common_constants.xacro"/>
     <xacro:include filename="$(find kuka_common)/urdf/common_materials.xacro"/>
-    <xacro:macro name="aip_cell" params="prefix">
+    <xacro:macro name="table" params="prefix">
         <link name="${prefix}table_link">
             <visual>
@@ -9,11 +9,4 @@
                 <geometry>
                     <mesh filename="package://aip_cell_description/meshes/aip_cell/visual/table0.001.stl" scale="0.001 0.001 0.001"/>
-                </geometry>
-                <xacro:material_kuka_ral_silver_gray/>
-            </visual>
-            <visual>
-                <origin xyz="0 0 0" rpy="0 0 0"/>
-                <geometry>
-                    <mesh filename="package://aip_cell_description/meshes/aip_cell/visual/Gestell.stl" scale="0.001 0.001 0.001"/>
                 </geometry>
                 <xacro:material_kuka_ral_silver_gray/>
@@ -25,12 +18,6 @@
                 </geometry>
             </collision>
-            <collision>
-                <origin xyz="0 0 0" rpy="0 0 0"/>
-                <geometry>
-                    <mesh filename="package://aip_cell_description/meshes/aip_cell/collision/Gestell.stl" scale="0.001 0.001 0.001"/>
-                </geometry>
-            </collision>
         </link>
-        <link name="${prefix}shelf">
+        <!-- <link name="${prefix}shelf">
             <visual>
                 <origin xyz="0 0 0" rpy="0 0 0"/>
@@ -46,5 +33,5 @@
                 </geometry>
             </collision>
-        </link>
+        </link> -->
         <link name="${prefix}ejector">
             <visual>
@@ -62,9 +49,9 @@
             </collision>
         </link>
-        <joint name="${prefix}joint_table-shelf" type="fixed">
+        <!-- <joint name="${prefix}joint_table-shelf" type="fixed">
             <parent link="${prefix}table_link"/>
             <child link="${prefix}shelf"/>
             <origin xyz="0.242 0.806 0.908" rpy="0 0 0"/>
-        </joint>
+        </joint> -->
     </xacro:macro>
 </robot>
